File: HVAB.kicad_sch (KiCad schematic)
At the start: 86 parts, among them J1 Conn_02x02_Top_Bottom, J2 Conn_02x02_Top_Bottom, J3 Conn_02x02_Top_Bottom, J4 Conn_02x02_Top_Bottom, J5 Conn_02x02_Top_Bottom, J6 Conn_02x03_Top_Bottom, Q1 2N7002K, Q2 SIHD6N80AE-GE3, SW3 SW_Nidec_CAS-120A1, U1 173010335, U2 TLV9302xPW, U3 INA186A3, U4 1779205341, U5 STM32C092FCP6, U6 LNK3294G, U7 TCLT1007, U8 SN65HVD234

Commit message: Delete text
Other:
- note removed: "CANVUAR ELS CONNECTORS (S'HAN DE TROBAR UNS DE HV) MIRAR SI PROTECCIO DE SORTIDES POSAR PTC (R13, R18) MIRAR QUINA POTENCIA S'HA DE POSAR PER RESITENCIES AMB LEDS A A LIMETACIO O SI POSAR UN ZENER"
Changed lines of the file:
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@@
-		)
-	)
-	(text "CANVUAR ELS CONNECTORS (S'HAN DE TROBAR UNS DE HV)\nMIRAR SI PROTECCIO DE SORTIDES POSAR PTC (R13, R18)\nMIRAR QUINA POTENCIA S'HA DE POSAR PER RESITENCIES AMB LEDS A A LIMETACIO O SI POSAR UN ZENER"
-		(exclude_from_sim no)
-		(at 355.092 179.578 0)
-		(effects
-			(font
-				(size 1.27 1.27)
-			)
 		)
 	)
